File: lab4/lab4.kicad_sch (KiCad schematic)
At the start: 15 parts, among them U1 74LS197, U2 74LS86, U3 74LS86, U4 74LS86

Commit message: update lab4
Parts:
- added C0, C1, C2: 10n, symbol Device:C
- added R10, R11, R12: 10, symbol Device:R
Connections:
- net G0: now also C0.1, R10.2; no longer U2.3
- net G1: now also C1.1, R11.2; no longer U3.3
- net G2: now also C2.1, R12.2; no longer U4.3
- net GND: now also C0.2, C1.2, C2.2
- new net: R11.1, U3.3
- new net: R10.1, U2.3
- new net: R12.1, U4.3
Other:
- moved on the sheet: R0, R1, R2, R3, R4, R5, R6, R7
